File: suite61pcb/suite61pcb.kicad_sch (KiCad schematic)
At the start: 0 parts

Commit message: update schematic
Parts:
- added D? (x28): 1N4148W, Diode_SMD:D_SOD-123, symbol Diode:1N4148W
- added JS?: joystick_switch, marbastlib-various:joystick_psp1000, symbol marbastlib-various:joystick_switch
- added SW? (x28): MX_SW_HS, marbastlib-mx:SW_MX_HS_1u, symbol marbastlib-mx:MX_SW_HS
- added SW?: RotaryEncoder_Switch, symbol Device:RotaryEncoder_Switch
- added U1: nice_nano, nice-nano-kicad-master:nice_nano, symbol nice_nano:nice_nano
Connections:
- new net: D?.2 (A), SW?.2 (x28)
