File: suite61pcb/suite61pcb.kicad_sch (KiCad schematic)
At the start: 98 parts, among them J1 FFC_Receiver, J2 Joystick_FFC, J3 Battery JST, J4 OLED, SW1 MX_SW_HS, SW10 MX_SW_HS, SW11 MX_SW_HS, SW12 MX_SW_HS, SW13 MX_SW_HS, SW14 MX_SW_HS, SW15 MX_SW_HS, SW16 MX_SW_HS, SW17 MX_SW_HS, SW18 MX_SW_HS, SW19 MX_SW_HS, SW2 MX_SW_HS, SW20 MX_SW_HS, SW21 MX_SW_HS, SW22 MX_SW_HS, SW23 MX_SW_HS, SW24 MX_SW_HS, SW25 MX_SW_HS, SW26 MX_SW_HS, SW27 MX_SW_HS, SW28 MX_SW_HS, SW29 MX_SW_HS, SW3 MX_SW_HS, SW30 MX_SW_HS, SW31 MX_SW_HS, SW32 MX_SW_HS, SW33 MX_SW_HS, SW34 MX_SW_HS, SW35 RotaryEncoder_Switch, SW36 Reset_Button, SW4 MX_SW_HS, SW5 MX_SW_HS, SW6 MX_SW_HS, SW7 MX_SW_HS, SW8 MX_SW_HS, SW9 MX_SW_HS, U1 nice_nano

Commit message: update pcb
Parts:
- removed J2: Joystick_FFC, marbastlib-various:joystick_switch, symbol Connector:Conn_01x05_Male
- removed JS1: Joycon_Joystick, suite61:2-way joystick switch, symbol marbastlib-various:joystick_switch
- SW2, SW29: footprint marbastlib-mx:SW_MX_HS_1u -> marbastlib-mx:SW_MX_HS_1.5u
- SW23: footprint marbastlib-mx:SW_MX_HS_1u -> marbastlib-mx:SW_MX_1.5u
- SW3: footprint marbastlib-mx:SW_MX_HS_1u -> marbastlib-mx:SW_MX_1.75u
- SW4, SW6: footprint marbastlib-mx:SW_MX_HS_1u -> suite61:SW_MX_P_2.25u
- SW7: footprint marbastlib-mx:SW_MX_HS_1u -> marbastlib-mx:SW_MX_1u
Changed lines of the file:
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@@
-    (stroke (width 0) (type default) (color 0 0 0 0))
-  )
-  (wire (pts (xy 115.57 162.56) (xy 115.57 167.64))
     (stroke (width 0) (type default) (color 0 0 0 0))
   )
@@
     (stroke (width 0) (type default) (color 0 0 0 0))
   )
-  (wire (pts (xy 114.3 165.1) (xy 118.11 165.1))
-    (stroke (width 0) (type default) (color 0 0 0 0))
-  )
   (wire (pts (xy 334.01 180.34) (xy 304.8 180.34))
     (stroke (width 0) (type default) (color 0 0 0 0))
@@
     (stroke (width 0) (type default) (color 0 0 0 0))
   )
-  (wire (pts (xy 118.11 162.56) (xy 118.11 165.1))
-    (stroke (width 0) (type default) (color 0 0 0 0))
-  )
   (wire (pts (xy 137.16 106.68) (xy 137.16 127))
     (stroke (width 0) (type default) (color 0 0 0 0))
@@
     (stroke (width 0) (type default) (color 0 0 0 0))
   )
-  (wire (pts (xy 125.73 167.64) (xy 115.57 167.64))
-    (stroke (width 0) (type default) (color 0 0 0 0))
-  )
   (wire (pts (xy 284.48 59.69) (xy 278.13 59.69))
     (stroke (width 0) (type default) (color 0 0 0 0))
@@
     (stroke (width 0) (type default) (color 0 0 0 0))
   )
-  (wire (pts (xy 114.3 160.02) (xy 118.11 160.02))
-    (stroke (width 0) (type default) (color 0 0 0 0))
-  )
   (wire (pts (xy 185.42 139.7) (xy 187.96 139.7))
     (stroke (width 0) (type default) (color 0 0 0 0))
@@
     (stroke (width 0) (type default) (color 0 0 0 0))
   )
-  (wire (pts (xy 125.73 152.4) (xy 114.3 152.4))
-    (stroke (width 0) (type default) (color 0 0 0 0))
-  )
   (wire (pts (xy 236.22 49.53) (xy 242.57 49.53))
     (stroke (width 0) (type default) (color 0 0 0 0))
   )
-  (wire (pts (xy 114.3 157.48) (xy 118.11 157.48))
-    (stroke (width 0) (type default) (color 0 0 0 0))
-  )
   (wire (pts (xy 78.74 78.74) (xy 88.9 78.74))
     (stroke (width 0) (type default) (color 0 0 0 0))
   )
-  (wire (pts (xy 115.57 162.56) (xy 114.3 162.56))
-    (stroke (width 0) (type default) (color 0 0 0 0))
-  )
   (wire (pts (xy 280.67 99.06) (xy 280.67 101.6))
     (stroke (width 0) (type default) (color 0 0 0 0))
@@
   )
   (wire (pts (xy 246.38 134.62) (xy 248.92 134.62))
-    (stroke (width 0) (type default) (color 0 0 0 0))
-  )
-  (wire (pts (xy 114.3 152.4) (xy 114.3 154.94))
     (stroke (width 0) (type default) (color 0 0 0 0))
   )
@@
     (property "Reference" "SW4" (id 0) (at 86.36 81.28 0))
     (property "Value" "MX_SW_HS" (id 1) (at 86.36 83.82 0))
-    (property "Footprint" "marbastlib-mx:SW_MX_HS_1u" (id 2) (at 86.36 88.9 0)
+    (property "Footprint" "suite61:SW_MX_P_2.25u" (id 2) (at 86.36 88.9 0)
       (effects (font (size 1.27 1.27)) hide)
     )
@@
     (property "Reference" "SW2" (id 0) (at 86.36 40.64 0))
     (property "Value" "MX_SW_HS" (id 1) (at 86.36 43.18 0))
-    (property "Footprint" "marbastlib-mx:SW_MX_HS_1u" (id 2) (at 86.36 48.26 0)
+    (property "Footprint" "marbastlib-mx:SW_MX_HS_1.5u" (id 2) (at 86.36 48.26 0)
       (effects (font (size 1.27 1.27)) hide)
     )
@@
     (property "Reference" "SW7" (id 0) (at 93.98 81.28 0))
     (property "Value" "MX_SW_HS" (id 1) (at 93.98 83.82 0))
-    (property "Footprint" "marbastlib-mx:SW_MX_HS_1u" (id 2) (at 93.98 88.9 0)
+    (property "Footprint" "marbastlib-mx:SW_MX_1u" (id 2) (at 93.98 88.9 0)
       (effects (font (size 1.27 1.27)) hide)
     )
@@
     )
   )
-  (symbol (lib_id "marbastlib-various:joystick_switch") (at 125.73 160.02 0) (unit 1)
-    (in_bom yes) (on_board yes) (fields_autoplaced)
-    (property "Reference" "JS1" (id 0) (at 132.08 158.7499 0)
-      (effects (font (size 1.27 1.27)) (justify left))
-    )
-    (property "Value" "Joycon_Joystick" (id 1) (at 132.08 161.2899 0)
-      (effects (font (size 1.27 1.27)) (justify left))
-    )
-    (property "Footprint" "suite61:2-way joystick switch" (id 2) (at 125.73 160.02 0)
-      (effects (font (size 1.27 1.27)) hide)
-    )
-    (property "Datasheet" "" (id 3) (at 125.73 160.02 0)
-      (effects (font (size 1.27 1.27)) hide)
-    )
-    (pin "1")
-    (pin "2")
-    (pin "3")
-    (pin "4")
-    (pin "5")
-  )
   (symbol (lib_id "marbastlib-mx:MX_SW_HS") (at 139.7 48.26 0) (unit 1)
     (in_bom yes) (on_board yes) (fields_autoplaced)
@@
     (pin "2")
   )
-  (symbol (lib_id "Connector:Conn_01x05_Male") (at 109.22 160.02 0) (unit 1)
-    (in_bom yes) (on_board yes)
-    (property "Reference" "J2" (id 0) (at 106.68 160.02 0))
-    (property "Value" "Joystick_FFC" (id 1) (at 111.76 167.64 0))
-    (property "Footprint" "marbastlib-various:joystick_switch" (id 2) (at 109.22 160.02 0)
-      (effects (font (size 1.27 1.27)) hide)
-    )
-    (property "Datasheet" "~" (id 3) (at 109.22 160.02 0)
-      (effects (font (size 1.27 1.27)) hide)
-    )
-    (pin "1")
-    (pin "2")
-    (pin "3")
-    (pin "4")
-    (pin "5")
-  )
   (symbol (lib_id "marbastlib-mx:MX_SW_HS") (at 104.14 109.22 0) (unit 1)
     (in_bom yes) (on_board yes) (fields_autoplaced)
@@
     (property "Reference" "SW29" (id 0) (at 156.21 121.92 0))
     (property "Value" "MX_SW_HS" (id 1) (at 156.21 124.46 0))
-    (property "Footprint" "marbastlib-mx:SW_MX_HS_1u" (id 2) (at 156.21 129.54 0)
+    (property "Footprint" "marbastlib-mx:SW_MX_HS_1.5u" (id 2) (at 156.21 129.54 0)
       (effects (font (size 1.27 1.27)) hide)
     )
@@
     (property "Reference" "SW23" (id 0) (at 139.7 121.92 0))
     (property "Value" "MX_SW_HS" (id 1) (at 139.7 124.46 0))
-    (property "Footprint" "marbastlib-mx:SW_MX_HS_1u" (id 2) (at 139.7 129.54 0)
+    (property "Footprint" "marbastlib-mx:SW_MX_1.5u" (id 2) (at 139.7 129.54 0)
       (effects (font (size 1.27 1.27)) hide)
     )
@@
     (property "Reference" "SW6" (id 0) (at 93.98 60.96 0))
     (property "Value" "MX_SW_HS" (id 1) (at 93.98 63.5 0))
-    (property "Footprint" "marbastlib-mx:SW_MX_HS_1u" (id 2) (at 93.98 68.58 0)
+    (property "Footprint" "suite61:SW_MX_P_2.25u" (id 2) (at 93.98 68.58 0)
       (effects (font (size 1.27 1.27)) hide)
     )
@@
     (property "Reference" "SW3" (id 0) (at 86.36 60.96 0))
     (property "Value" "MX_SW_HS" (id 1) (at 86.36 63.5 0))
-    (property "Footprint" "marbastlib-mx:SW_MX_HS_1u" (id 2) (at 86.36 68.58 0)
+    (property "Footprint" "marbastlib-mx:SW_MX_1.75u" (id 2) (at 86.36 68.58 0)
       (effects (font (size 1.27 1.27)) hide)
     )
@@
       (reference "J1") (unit 1) (value "FFC_Receiver") (footprint "LIB_503480-0500:5034800500")
     )
-    (path "/5b0cb434-3114-453b-9a98-5306037bebb3"
-      (reference "J2") (unit 1) (value "Joystick_FFC") (footprint "marbastlib-various:joystick_switch")
-    )
     (path "/9019aa46-e007-4a20-a52f-6b687cc5d79f"
       (reference "J3") (unit 1) (value "Battery JST") (footprint "Connector_JST:JST_EH_B2B-EH-A_1x02_P2.50mm_Vertical")
@@
       (reference "JP8") (unit 1) (value "Jumper_NO_Small") (footprint "suite61:jumper")
     )
-    (path "/59f3f8c3-a02a-45e6-b943-5a967aac25b3"
-      (reference "JS1") (unit 1) (value "Joycon_Joystick") (footprint "suite61:2-way joystick switch")
-    )
     (path "/a149b419-122d-4faa-866a-fc943963345c"
       (reference "LED1") (unit 1) (value "SK6812MINI-E") (footprint "marbastlib-various:LED_6028R")
@@
     )
     (path "/418d1146-c9a7-43a9-85f2-18c7980c093e"
-      (reference "SW2") (unit 1) (value "MX_SW_HS") (footprint "marbastlib-mx:SW_MX_HS_1u")
+      (reference "SW2") (unit 1) (value "MX_SW_HS") (footprint "marbastlib-mx:SW_MX_HS_1.5u")
     )
     (path "/fb078fd2-8e59-4e51-991f-89db2c1094aa"
-      (reference "SW3") (unit 1) (value "MX_SW_HS") (footprint "marbastlib-mx:SW_MX_HS_1u")
+      (reference "SW3") (unit 1) (value "MX_SW_HS") (footprint "marbastlib-mx:SW_MX_1.75u")
     )
     (path "/19fc4a23-cdc3-47fa-9888-fe386efd8b63"
-      (reference "SW4") (unit 1) (value "MX_SW_HS") (footprint "marbastlib-mx:SW_MX_HS_1u")
+      (reference "SW4") (unit 1) (value "MX_SW_HS") (footprint "suite61:SW_MX_P_2.25u")
     )
     (path "/70a6584d-b631-4264-a991-0777c61d5600"
@@
     )
     (path "/a21fb532-93aa-412a-a737-962b3a2e38ec"
-      (reference "SW6") (unit 1) (value "MX_SW_HS") (footprint "marbastlib-mx:SW_MX_HS_1u")
+      (reference "SW6") (unit 1) (value "MX_SW_HS") (footprint "suite61:SW_MX_P_2.25u")
     )
     (path "/526f7ea9-c956-427f-a7e4-eeb006656c52"
-      (reference "SW7") (unit 1) (value "MX_SW_HS") (footprint "marbastlib-mx:SW_MX_HS_1u")
+      (reference "SW7") (unit 1) (value "MX_SW_HS") (footprint "marbastlib-mx:SW_MX_1u")
     )
     (path "/4815b6bf-93af-4cde-b040-ee1136493752"
@@
     )
     (path "/9e1db182-01ca-4a14-aa90-e89b165ce1a6"
-      (reference "SW23") (unit 1) (value "MX_SW_HS") (footprint "marbastlib-mx:SW_MX_HS_1u")
+      (reference "SW23") (unit 1) (value "MX_SW_HS") (footprint "marbastlib-mx:SW_MX_1.5u")
     )
     (path "/b8ce77b3-493b-4a7f-8ffe-ac0ee2951038"
@@
     )
     (path "/63603601-8efa-417a-8658-83201e179789"
-      (reference "SW29") (unit 1) (value "MX_SW_HS") (footprint "marbastlib-mx:SW_MX_HS_1u")
+      (reference "SW29") (unit 1) (value "MX_SW_HS") (footprint "marbastlib-mx:SW_MX_HS_1.5u")
     )
     (path "/a89d72ac-264f-4298-ab26-0c18d63285b3"

Commit message: update pcb and add keebio submod
Parts:
- added SW36: MX_SW_HS, marbastlib-mx:SW_MX_HS_1u, symbol marbastlib-mx:MX_SW_HS
- SW13: renamed from SW3; value MX_SW_HS -> MX_SW
- SW14: renamed from SW6; value MX_SW_HS -> MX_SW
- SW21: renamed from SW4; value MX_SW_HS -> MX_SW
- SW22: renamed from SW7; value MX_SW_HS -> MX_SW
- renumbered D18 to D10, D24 to D11, D31 to D12, D3 to D13, D8 to D14, D14 to D15, D19 to D16, D25 to D17, D32 to D18, D4 to D19, D6 to D2, D9 to D20, D15 to D21, D20 to D22, D26 to D23, D33 to D24, D5 to D25, D10 to D26, D16 to D27, D21 to D28, D27 to D29, D12 to D3, D34 to D30, D22 to D31, D28 to D32, D11 to D33, D29 to D34, D17 to D4, D23 to D5, D30 to D6, D2 to D7, D7 to D8, D13 to D9, J3 to J1, J4 to J2, J1 to J3, SW19 to SW10, SW25 to SW11, SW31 to SW12, SW10 to SW15, SW15 to SW16, SW20 to SW17, SW26 to SW18, SW32 to SW19, SW8 to SW2, SW36 to SW20, SW11 to SW23, SW16 to SW24, SW21 to SW25, SW27 to SW26, SW33 to SW27, SW5 to SW28, SW12 to SW29, SW13 to SW3, SW17 to SW30, SW22 to SW31, SW28 to SW32, SW34 to SW33, SW23 to SW34, SW29 to SW35, SW35 to SW37, SW18 to SW4, SW24 to SW5, SW30 to SW6, SW2 to SW7, SW9 to SW8, SW14 to SW9
Connections:
- net col0: now also SW36.1
- net at D34.2 (A), SW37.S1: now also SW36.2
Other:
- moved on the sheet: SW37

Commit message: update pcb and schematic
Parts:
- added C1, C2: 100nF, Capacitor_SMD:C_0805_2012Metric, symbol Device:C_Small
- added D31: 1N4148W, Diode_SMD:D_SOD-123, symbol Diode:1N4148W
- J1: footprint Connector_JST:JST_EH_B2B-EH-A_1x02_P2.50mm_Vertical -> Connector_JST:JST_EH_S2B-EH_1x02_P2.50mm_Horizontal
- LED1, LED2, LED3, LED4, LED5, LED6: footprint marbastlib-various:LED_6028R -> LED_SMD:LED_SK6812MINI_PLCC4_3.5x3.5mm_P1.75mm
- SW37: footprint marbastlib-various:ROT_Alps_EC11E-Switch -> Keebio-Parts:RotaryEncoder_EC11
- renumbered D31 to D32, D32 to D33, D33 to D34, D34 to D35
Connections:
- net BATTERY: now also S1.B1 (COM); no longer S1.C1 (NO)
- net Enc0: now also C2.2
- net Enc1: now also C1.1
- net GND: now also C1.2, C2.1
- net VCC: now also J3.1 (Pin_1), D31.1 (K)
- net col0: now also SW36.2, SW37.S1; no longer SW36.1, SW37.S2
- net col3: now also D31.2 (A); no longer J3.1 (Pin_1)
- net row5: now also D32.1 (K), D33.1 (K), D35.1 (K)
- net at J1.2 (Pin_2): now also S1.C1 (NO); no longer S1.B1 (COM)
- new net: D34.2 (A), J3.3 (Pin_3)
- new net: D35.2 (A), SW36.1, SW37.S2
Other:
- moved on the sheet: D34, J1, J3, SW37
