File: suite61pcb/LIB_MSK12C02/suite61pcbleft.kicad_sch (KiCad schematic)
At the start: 79 parts, among them J1 FFC_Receiver, J2 Joystick_FFC, J3 Battery JST, J4 OLED, SW1 MX_SW_HS, SW10 MX_SW_HS, SW11 MX_SW_HS, SW12 MX_SW_HS, SW13 MX_SW_HS, SW14 MX_SW_HS, SW15 MX_SW_HS, SW16 MX_SW_HS, SW17 MX_SW_HS, SW18 MX_SW_HS, SW19 MX_SW_HS, SW2 MX_SW_HS, SW20 MX_SW_HS, SW21 MX_SW_HS, SW22 MX_SW_HS, SW23 MX_SW_HS, SW24 MX_SW_HS, SW25 MX_SW_HS, SW26 MX_SW_HS, SW27 MX_SW_HS, SW28 MX_SW_HS, SW29 RotaryEncoder_Switch, SW3 MX_SW_HS, SW30 Reset_Button, SW4 MX_SW_HS, SW5 MX_SW_HS, SW6 MX_SW_HS, SW7 MX_SW_HS, SW8 MX_SW_HS, SW9 MX_SW_HS, U1 nice_nano

Commit message: create left pcb schematic
Parts:
- removed TH1, TH2, TH3, TH4, TH5: HOLE, MountingHole:MountingHole_3.7mm, symbol keebio:Hole
- J?: renamed from J2; footprint marbastlib-various:joystick_switch -> (none)
- J?: renamed from J1; footprint LIB_503480-0500:5034800500 -> (none)
- J?: renamed from J3; footprint Connector_JST:JST_EH_B2B-EH-A_1x02_P2.50mm_Vertical -> (none)
- J?: renamed from J4; footprint Connector_PinHeader_2.00mm:PinHeader_1x04_P2.00mm_Vertical -> (none)
- S?: renamed from S1; footprint LIB_MSK12C02:MSK12C02 -> MSK12C02
- SW?: renamed from SW30; footprint Button_Switch_SMD:SW_Push_1P1T_NO_CK_KMR2 -> (none)
- SW?: renamed from SW29; footprint marbastlib-various:ROT_Alps_EC11E-Switch -> (none)
- renumbered D2 to D?, D3 to D?, D23 to D?, D8 to D?, D17 to D?, D4 to D?, D28 to D?, D1 to D?, D16 to D?, D24 to D?, D29 to D?, D15 to D?, D10 to D?, D19 to D?, D21 to D?, D22 to D?, D5 to D?, D9 to D?, D12 to D?, D25 to D?, D26 to D?, D14 to D?, D11 to D?, D7 to D?, D18 to D?, D27 to D?, D6 to D?, D20 to D?, D13 to D?, JP1 to JP?, JP8 to JP?, JP7 to JP?, JP4 to JP?, JP2 to JP?, JP3 to JP?, JP5 to JP?, JP6 to JP?, JS1 to JS?, SW8 to SW?, SW4 to SW?, SW22 to SW?, SW24 to SW?, SW2 to SW?, SW6 to SW?, SW26 to SW?, SW12 to SW?, SW17 to SW?, SW16 to SW?, SW10 to SW?, SW1 to SW?, SW5 to SW?, SW19 to SW?, SW18 to SW?, SW7 to SW?, SW25 to SW?, SW28 to SW?, SW20 to SW?, SW21 to SW?, SW27 to SW?, SW15 to SW?, SW13 to SW?, SW11 to SW?, SW14 to SW?, SW23 to SW?, SW9 to SW?, SW3 to SW?
